File: PCB/sponka.kicad_pcb (KiCad board)
At the start: 2 copper layers, 0 parts

Commit message: Made first PCB
Parts:
- added BAT: Conn_01x02_Socket, Connector_PinHeader_2.54mm:PinHeader_1x02_P2.54mm_Horizontal, F.Cu at (182.6, 105.9)
- added C1: 100nF, Capacitor_SMD:C_0402_1005Metric, F.Cu at (172.2, 99.8)
- added C2: 10uF, Capacitor_SMD:C_0402_1005Metric, F.Cu at (114.8, 102.9)
- added C3: 10uF, Capacitor_SMD:C_0402_1005Metric, F.Cu at (112.6, 99.6)
- added C4: 100n, Capacitor_SMD:C_0402_1005Metric, F.Cu at (114.8, 101.7)
- added C5: 100nF, Capacitor_SMD:C_0402_1005Metric, F.Cu at (172.3, 103.7)
- added CHRG: LED, LED_SMD:LED_0603_1608Metric, F.Cu at (116.3, 96.6)
- added D1: WS2812B, LED_SMD:LED_WS2812B_PLCC4_5.0x5.0mm_P3.2mm, F.Cu at (166.7, 101.3)
- added D2: WS2812B, LED_SMD:LED_WS2812B_PLCC4_5.0x5.0mm_P3.2mm, F.Cu at (158.7, 101.3)
- added D3: WS2812B, LED_SMD:LED_WS2812B_PLCC4_5.0x5.0mm_P3.2mm, F.Cu at (150.7, 101.3)
- added D4: WS2812B, LED_SMD:LED_WS2812B_PLCC4_5.0x5.0mm_P3.2mm, F.Cu at (142.7, 101.3)
- added D5: WS2812B, LED_SMD:LED_WS2812B_PLCC4_5.0x5.0mm_P3.2mm, F.Cu at (134.7, 101.3)
- added D6: WS2812B, LED_SMD:LED_WS2812B_PLCC4_5.0x5.0mm_P3.2mm, F.Cu at (126.7, 101.3)
- added J2: USB_C_Receptacle_USB2.0_14P, Connector_USB:USB_C_Receptacle_G-Switch_GT-USB-7010ASV, F.Cu at (105.1, 101.4)
- added MCU: CH32V003FxUx, Package_DFN_QFN:QFN-20-1EP_3x3mm_P0.4mm_EP1.65x1.65mm_ThermalVias, F.Cu at (174.8, 98.8)
- added R1: 2.2k, Resistor_SMD:R_0402_1005Metric, F.Cu at (116.5, 98.6)
- added R2: 5k, Resistor_SMD:R_0402_1005Metric, F.Cu at (110.5, 97.0)
- added R3: 5.1k, Resistor_SMD:R_0402_1005Metric, F.Cu at (110.5, 99.6)
- added R4: 5.1k, Resistor_SMD:R_0402_1005Metric, F.Cu at (110.5, 103.9)
- added R5: 33, Resistor_SMD:R_0402_1005Metric, F.Cu at (111.9, 100.6)
- added R6: 33, Resistor_SMD:R_0402_1005Metric, F.Cu at (111.9, 102.1)
- added R7: 470k, Resistor_SMD:R_0402_1005Metric, F.Cu at (120.4, 104.3)
- added R8: 470k, Resistor_SMD:R_0402_1005Metric, F.Cu at (121.4, 104.3)
- added RESET: SW_Push, Button_Switch_SMD:SW_SPST_B3U-1000P-B, F.Cu at (172.2, 105.9)
- added STDBY: LED, LED_SMD:LED_0603_1608Metric, F.Cu at (117.8, 96.6)
- added SW: SW_SPDT, Button_Switch_SMD:SW_SPDT_PCM12, F.Cu at (115.5, 105.8)
- added SWD: Conn_01x03_Pin, Connector_PinHeader_2.54mm:PinHeader_1x03_P2.54mm_Vertical, F.Cu at (179.0, 101.5)
- added U2: TP4057, Package_TO_SOT_SMD:TSOT-23-6, F.Cu at (113.1, 97.4)
- added U3: AP2127K-3.3, Package_TO_SOT_SMD:SOT-23-5, F.Cu at (117.5, 101.1)
Routing:
- net Net-(J3-Pin_2): track 0.00 -> 80.4 mm, vias 0 -> 2
- net +3V3: track 0.00 -> 79.9 mm
- net GND: track 0.00 -> 76.1 mm, vias 0 -> 8
- net /Power management/USB_DN: track 0.00 -> 70.5 mm, vias 0 -> 2
- net /Power management/USB_DP: track 0.00 -> 69.2 mm, vias 0 -> 2
- net /Power management/BATT_DIV: track 0.00 -> 58.0 mm, vias 0 -> 2
- net /Power management/VBUS: track 0.00 -> 17.8 mm, vias 0 -> 2
- net Net-(D1-DOUT): track 0.00 -> 14.3 mm
- net Net-(D3-DOUT): track 0.00 -> 14.3 mm
- net Net-(D2-DOUT): track 0.00 -> 14.3 mm
- net Net-(D4-DOUT): track 0.00 -> 14.3 mm
- net Net-(D5-DOUT): track 0.00 -> 14.3 mm
- net /LED Row/Row_DIN: track 0.00 -> 11.6 mm, vias 0 -> 2
- net Net-(U1-PD7): track 0.00 -> 9.39 mm, vias 0 -> 2
- net Net-(SW1-C): track 0.00 -> 7.47 mm
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- added copper zone on B.Cu, net GND
Other:
- board outline added: 87.1 x 13.3 mm

Commit message: PCB V2
Parts:
- removed BAT: Conn_01x02_Socket, Connector_PinHeader_2.54mm:PinHeader_1x02_P2.54mm_Horizontal
- removed CHRG, STDBY: LED, LED_SMD:LED_0603_1608Metric
- removed MCU: CH32V003FxUx, Package_DFN_QFN:QFN-20-1EP_3x3mm_P0.4mm_EP1.65x1.65mm_ThermalVias
- removed RESET: SW_Push, Button_Switch_SMD:SW_SPST_B3U-1000P-B
- removed SW: SW_SPDT, Button_Switch_SMD:SW_SPDT_PCM12
- removed SWD: Conn_01x03_Pin, Connector_PinHeader_2.54mm:PinHeader_1x03_P2.54mm_Vertical
- added D_CHRG1: LED, LED_SMD:LED_0603_1608Metric, F.Cu at (116.9, 96.5)
- added D_STDBY1: LED, LED_SMD:LED_0603_1608Metric, F.Cu at (116.9, 98.0)
- added J1: Conn_01x03_Pin, sponka:pogo_pins, F.Cu at (144.5, 106.2)
- added J3: Conn_01x02_Socket, Connector_PinHeader_2.54mm:PinHeader_1x02_P2.54mm_Horizontal, F.Cu at (183.2, 105.8)
- added SW1: SW_Push, Button_Switch_SMD:SW_SPST_B3U-1000P-B, F.Cu at (120.1, 106.0)
- added SW2: SW_SPDT, Button_Switch_SMD:SW_SPDT_PCM12, F.Cu at (174.0, 105.8)
- added U1: CH32V003FxUx, Package_DFN_QFN:QFN-20-1EP_3x3mm_P0.4mm_EP1.65x1.65mm_ThermalVias, F.Cu at (117.0, 102.0)
- C2: value 10uF -> 100nF
- C4: value 100n -> 10uF
- C5: value 100nF -> 100n
- R1: value 2.2k -> 5.1k
- R2: value 5k -> 5.1k
- R3, R4: value 5.1k -> 33
- R5: value 33 -> 2.2k
- R6: value 33 -> 5k
- moved U3 62.2 mm to (179.7, 101.3)
- moved R7 60.0 mm to (180.4, 105.0), turned to 180 degrees
- moved R8 59.0 mm to (180.4, 106.0), turned to 0 degrees
- moved C1 52.3 mm to (120.0, 102.9), turned to 0 degrees
- moved D1 40.7 mm to (126.0, 101.0), turned to 0 degrees
- moved D6 39.4 mm to (166.0, 101.0), turned to 0 degrees
- moved D2 24.7 mm to (134.0, 101.0), turned to 0 degrees
- moved D5 23.4 mm to (158.0, 101.0), turned to 0 degrees
- moved D3 8.66 mm to (142.0, 101.0), turned to 0 degrees
- moved D4 7.36 mm to (150.0, 101.0), turned to 0 degrees
- moved R1 7.03 mm to (109.5, 99.7), turned to -90 degrees
- moved C4 6.54 mm to (109.5, 97.8), turned to -90 degrees
- moved R2 6.52 mm to (109.5, 103.5), turned to 90 degrees
- moved R6 5.97 mm to (114.7, 96.8), turned to -90 degrees
- moved C5 5.61 mm to (177.5, 101.6), turned to -90 degrees
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Connections:
- C2 pad 2: Net-(J3-Pin_2) -> Net-(U1-PD7)
- C4 pad 1: +3V3 -> GND
- C4 pad 2: GND -> Net-(J3-Pin_2)
- C5 pad 1: GND -> +3V3
- C5 pad 2: Net-(U1-PD7) -> GND
- R1 pad 1: /Power management/VBUS -> GND
- R1 pad 2: Net-(D46-A) -> Net-(J2-CC1)
- R2 pad 1: Net-(U2-PROG) -> GND
- R2 pad 2: GND -> Net-(J2-CC2)
- R3 pad 1: GND -> /Power management/USB_DN
- R3 pad 2: Net-(J2-CC1) -> Net-(J2-D--PadA7)
- R4 pad 1: GND -> /Power management/USB_DP
- R4 pad 2: Net-(J2-CC2) -> Net-(J2-D+-PadA6)
- R5 pad 1: /Power management/USB_DN -> /Power management/VBUS
- R5 pad 2: Net-(J2-D--PadA7) -> Net-(D_CHRG1-A)
- R6 pad 1: /Power management/USB_DP -> Net-(U2-PROG)
- R6 pad 2: Net-(J2-D+-PadA6) -> GND
Routing:
- net /Power management/USB_DN: track 70.5 -> 4.79 mm, vias 2 -> 0
- net /Power management/USB_DP: track 69.2 -> 4.54 mm, vias 2 -> 0
- net Net-(J1-Pin_2): track 3.16 -> 31.7 mm, vias 0 -> 2
- net +3V3: track 79.9 -> 96.8 mm
- net /Power management/BATT_DIV: track 58.0 -> 70.1 mm
- net Net-(D_CHRG1-A): track 0.00 -> 4.07 mm
- net Net-(U2-PROG): track 4.79 -> 1.35 mm, vias 2 -> 0
- net Net-(D46-A): track 3.04 -> 0.00 mm
- net Net-(D_CHRG1-K): track 4.60 -> 7.63 mm, vias 0 -> 2
- net Net-(J3-Pin_2): track 80.4 -> 83.4 mm, vias 2 -> 4
- net Net-(U1-PD7): track 9.39 -> 6.61 mm, vias 2 -> 0
- net Net-(SW2-C): track 7.47 -> 10.1 mm
- net GND: track 76.1 -> 74.2 mm, vias 8 -> 10
- net /Power management/VBUS: track 17.8 -> 19.4 mm, vias 2 -> 0
- net Net-(D_STDBY1-K): track 4.22 -> 3.14 mm
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Other:
- board text added: "USB-C"

Commit message: New PCB design
Parts:
- moved J3 11.7 mm to (176.2, 96.4), turned to 0 degrees
- moved SW2 8.40 mm to (182.4, 105.8)
- moved R7 4.37 mm to (176.0, 104.7)
- moved R8 4.37 mm to (176.0, 105.7)
- moved C5 4.32 mm to (173.4, 103.0), turned to 90 degrees
- moved U3 3.96 mm to (175.9, 102.5), turned to 180 degrees
Routing:
- net +3V3: track 96.8 -> 92.4 mm
- net Net-(J3-Pin_2): track 83.4 -> 79.1 mm, vias 4 -> 2
- net Net-(SW2-C): track 10.1 -> 14.0 mm
- net /Power management/BATT_DIV: track 70.1 -> 66.9 mm
- net GND: track 74.2 -> 72.2 mm
Other:
- board text added: "+"
- board text added: "-"
- board text added: "BAT"
- board text added: "CHRG"
- board text added: "La Sponka"
- board text added: "RESET"
- board text added: "RISC-V MCU"
- board text added: "STBY"
- board text added: "SWITCH"
- board text added: "WS2812B"
- board text added: "by Vesek"
- board text added: "↓"

Commit message: New PCB revision
Parts:
- J3: footprint Connector_PinHeader_2.54mm:PinHeader_1x02_P2.54mm_Horizontal -> sponka:HDR-SMD_2P-P2.54-H-M-W13.3-N
- moved J3 8.96 mm to (185.0, 97.8), turned to -90 degrees
- moved SW2 0.45 mm to (181.9, 105.8)
- moved C5 0.42 mm to (173.0, 103.0)
- moved U3 0.42 mm to (175.5, 102.5)
Routing:
- net Net-(J3-Pin_2): track 79.1 -> 84.3 mm
- net GND: track 72.2 -> 75.6 mm, vias 10 -> 11
- net +3V3: track 92.4 -> 91.3 mm
- net Net-(SW2-C): track 14.0 -> 13.3 mm
Other:
- outline, holes or cut-outs redrawn
- board text added: "Návod"

Commit message: Probably the final update
Parts:
- added J4: Conn_01x05_Pin, sponka:pogo_pins_1_5, F.Cu at (129.2, 96.5)
- added R9: 5,1k, Resistor_SMD:R_0402_1005Metric, F.Cu at (113.5, 101.0)
- J1: footprint sponka:pogo_pins -> sponka:pogo_pins_1_3
- moved C1 0.20 mm to (120.2, 102.9)
- moved C2 0.10 mm to (120.0, 103.8)
Connections:
- U1 pad 13: unconnected-(U1-PC6-Pad13) -> /LED Row/Row_DIN
- U1 pad 16: unconnected-(U1-PD2-Pad16) -> /DPU
- U1 pad 7: /LED Row/Row_DIN -> /TX
- U1 pad 8: unconnected-(U1-PC1-Pad8) -> /RX/SDA
- U1 pad 9: unconnected-(U1-PC2-Pad9) -> /RTS/SCL
Routing:
- net /TX: track 0.00 -> 16.5 mm
- net /RX/SDA: track 0.00 -> 13.8 mm
- net /RTS/SCL: track 0.00 -> 12.9 mm
- net +3V3: track 91.3 -> 93.7 mm
- net GND: track 75.6 -> 77.4 mm, vias 11 -> 12
- net Net-(J1-Pin_2): track 31.9 -> 33.7 mm
- net /DPU: track 0.00 -> 1.57 mm
- net /Power management/USB_DN: track 4.79 -> 5.83 mm
- net /LED Row/Row_DIN: track 11.9 -> 12.8 mm
- net Net-(J3-Pin_2): track 84.3 -> 83.5 mm
Other:
- board text added: "BTN"
- board text added: "I2C"
- board text added: "R"
- board text added: "RS"
- board text added: "SCL"
- board text added: "SDA"
- board text added: "SWIO"
- board text added: "T"
- board text added: "UART"
- board text removed: "RESET"
