File: PCB/array.kicad_sch (KiCad schematic)
At the start: 9 parts

Commit message: Made first PCB
Parts:
- removed D1, D2, D3, D4, D5, D6, D7, D8, D9: WS2812B-2020, LED_SMD:LED_WS2812B-2020_PLCC4_2.0x2.0mm, symbol LED:WS2812B-2020
- added D1, D2, D3, D4, D5, D6: WS2812B, LED_SMD:LED_WS2812B_PLCC4_5.0x5.0mm_P3.2mm, symbol LED:WS2812B
Connections:
- net +3V3: now also D1.1 (VDD), D2.1 (VDD), D3.1 (VDD), D4.1 (VDD), D5.1 (VDD), D6.1 (VDD)
- net GND: now also D1.3 (VSS), D2.3 (VSS), D3.3 (VSS), D4.3 (VSS), D5.3 (VSS), D6.3 (VSS)
- net Row_DIN: now also D1.4 (DIN)
- new net: D2.2 (DOUT), D3.4 (DIN)
- new net: D1.2 (DOUT), D2.4 (DIN)
- new net: D3.2 (DOUT), D4.4 (DIN)
- new net: D5.2 (DOUT), D6.4 (DIN)
- new net: D4.2 (DOUT), D5.4 (DIN)

Commit message: Made smol :) Anyway, this is just WIP, still working on it
Parts:
- removed D1, D2, D3, D4, D5, D6: WS2812B, LED_SMD:LED_WS2812B_PLCC4_5.0x5.0mm_P3.2mm, symbol LED:WS2812B
- added LED1, LED2, LED3, LED4, LED5, LED6: WS2812B-MINI, sponka:LED-SMD_4P-L3.5-W3.5-TL_WS2812B, symbol sponka:WS2812B-MINI
Connections:
- net +3V3: now also LED1.1 (VDD), LED2.1 (VDD), LED3.1 (VDD), LED4.1 (VDD), LED5.1 (VDD), LED6.1 (VDD)
- net GND: now also LED1.3 (VSS), LED2.3 (VSS), LED3.3 (VSS), LED4.3 (VSS), LED5.3 (VSS), LED6.3 (VSS)
- net Row_DIN: now also LED1.4 (DIN)
- new net: LED2.2 (DOUT), LED3.4 (DIN)
- new net: LED1.2 (DOUT), LED2.4 (DIN)
- new net: LED5.2 (DOUT), LED6.4 (DIN)
- new net: LED4.2 (DOUT), LED5.4 (DIN)
- new net: LED3.2 (DOUT), LED4.4 (DIN)

Commit message: New design WIP
Parts:
- removed LED6: WS2812B-MINI, sponka:LED-SMD_4P-L3.5-W3.5-TL_WS2812B, symbol sponka:WS2812B-MINI
Changed lines of the file:
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@@
 	(paper "A4")
 	(junction
-		(at 92.71 93.98)
-		(diameter 0)
-		(color 0 0 0 0)
-	)
-	(junction
 		(at 97.79 78.74)
 		(diameter 0)
@@
 	)
 	(junction
-		(at 72.39 78.74)
-		(diameter 0)
-		(color 0 0 0 0)
-	)
-	(junction
 		(at 143.51 93.98)
 		(diameter 0)
@@
 	(wire
 		(pts
-			(xy 68.58 93.98) (xy 92.71 93.98)
-		)
-		(stroke
-			(width 0)
-			(type default)
-		)
-	)
-	(wire
-		(pts
 			(xy 146.05 87.63) (xy 148.59 87.63)
 		)
@@
 	(wire
 		(pts
-			(xy 92.71 93.98) (xy 118.11 93.98)
+			(xy 68.58 93.98) (xy 118.11 93.98)
 		)
 		(stroke
@@
 	(wire
 		(pts
-			(xy 95.25 87.63) (xy 97.79 87.63)
-		)
-		(stroke
-			(width 0)
-			(type default)
-		)
-	)
-	(wire
-		(pts
-			(xy 72.39 85.09) (xy 72.39 78.74)
-		)
-		(stroke
-			(width 0)
-			(type default)
-		)
-	)
-	(wire
-		(pts
 			(xy 195.58 87.63) (xy 195.58 93.98)
 		)
@@
 	(wire
 		(pts
-			(xy 92.71 87.63) (xy 92.71 93.98)
-		)
-		(stroke
-			(width 0)
-			(type default)
-		)
-	)
-	(wire
-		(pts
 			(xy 148.59 78.74) (xy 148.59 85.09)
 		)
@@
 	(wire
 		(pts
-			(xy 72.39 78.74) (xy 97.79 78.74)
-		)
-		(stroke
-			(width 0)
-			(type default)
-		)
-	)
-	(wire
-		(pts
-			(xy 95.25 85.09) (xy 95.25 87.63)
-		)
-		(stroke
-			(width 0)
-			(type default)
-		)
-	)
-	(wire
-		(pts
 			(xy 171.45 85.09) (xy 171.45 87.63)
 		)
@@
 	(wire
 		(pts
-			(xy 68.58 78.74) (xy 72.39 78.74)
-		)
-		(stroke
-			(width 0)
-			(type default)
-		)
-	)
-	(wire
-		(pts
-			(xy 92.71 85.09) (xy 95.25 85.09)
+			(xy 68.58 78.74) (xy 97.79 78.74)
 		)
 		(stroke
@@
 					(unit 1)
 				)
-			)
-		)
-	)
-	(symbol
-		(lib_id "sponka:WS2812B-MINI")
-		(at 82.55 86.36 0)
-		(unit 1)
-		(exclude_from_sim no)
-		(in_bom yes)
-		(on_board yes)
-		(dnp no)
-		(fields_autoplaced yes)
-		(property "Reference" "LED6"
-			(at 82.55 77.47 0)
-			(effects
-				(font
-					(size 1.27 1.27)
-				)
-			)
-		)
-		(property "Value" "WS2812B-MINI"
-			(at 82.55 80.01 0)
-			(effects
-				(font
-					(size 1.27 1.27)
-				)
-			)
-		)
-		(property "Footprint" "sponka:LED-SMD_4P-L3.5-W3.5-TL_WS2812B"
-			(at 82.55 95.25 0)
-			(effects
-				(font
-					(size 1.27 1.27)
-				)
-				(hide yes)
-			)
-		)
-		(property "Datasheet" "https://lcsc.com/product-detail/Light-Emitting-Diodes-LED_Worldsemi-WS2812B-Mini_C527089.html"
-			(at 82.55 97.79 0)
-			(effects
-				(font
-					(size 1.27 1.27)
-				)
-				(hide yes)
-			)
-		)
-		(property "Description" ""
-			(at 82.55 86.36 0)
-			(effects
-				(font
-					(size 1.27 1.27)
-				)
-				(hide yes)
-			)
-		)
-		(property "LCSC Part" "C527089"
-			(at 82.55 100.33 0)
-			(effects
-				(font
-					(size 1.27 1.27)
-				)
-				(hide yes)
-			)
-		)
-		(pin "2"
-		)
-		(pin "4"
-		)
-		(pin "3"
-		)
-		(pin "1"
-		)
-		(instances
-			(project ""
-				(path "/cd633adc-49f5-4b4f-8d72-c74316356641/059eed50-6267-4cf5-8368-3ab59d67dd86"
-					(reference "LED6")
-					(unit 1)
-				)
